File: Rev.0/CAD/39c3PCBLEDC100R_Rev.0.kicad_pcb (KiCad board)
At the start: 2 copper layers, 100 x 100 mm, 26 parts, among them Q2 ZVNL110A, U1 WeMos_D1_mini

Commit message: First commit of the updated Design files
Parts:
- renumbered H1 to +5V, Q2 to Q1
Connections:
- Q1 pad 1: Net-(Q2-S) -> (no net)
- R2 pad 2: Net-(Q2-S) -> Net-(Q1-S)
- U1 pad 11: Net-(Q2-S) -> Net-(Q1-S)
Routing:
- net Net-(Q2-S): track 56.0 -> 0.00 mm
- net Net-(Q1-S): track 0.00 -> 56.0 mm
Other:
- board text added: "Hackers should be judged by their hacking, not bogus criteria such as degrees, age, race, or position"
- board text removed: "Mistrust authority - promote decentralization."

Commit message: Added files for production & fixed some minor errors on the silkscreen
Parts:
- added REF**: 39c3_Text, Logo:39c3_Text, B.Cu at (150.0, 100.0)
- added SW1: SW_SPST, Button_Switch_THT:SW_TH_Tactile_Omron_B3F-102x, B.Cu at (180.0, 127.6)
Connections:
- Q1 pad 1: (no net) -> Net-(Q1-S)
- U1 pad 12: unconnected-(U1-D3-Pad12) -> Net-(SW1-A)
Routing:
- net Net-(SW1-A): track 0.00 -> 46.6 mm
