File: Rev.0/CAD/39c3PCBLEDC100R_Rev.0.kicad_sch (KiCad schematic)
At the start: 22 parts, among them Q2 ZVNL110A, U1 WeMos_D1_mini

Commit message: First commit of the updated Design files
Parts:
- renumbered Q2 to Q1
Changed lines of the file:
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@@
 		(dnp no)
 		(fields_autoplaced yes)
-		(property "Reference" "Q2"
+		(property "Reference" "Q1"
 			(at 140.97 102.87 90)
 			(effects
@@
 			(project ""
 				(path "/4acc92b7-ae78-4f6f-8f1d-403b41b8ff51"
-					(reference "Q2")
+					(reference "Q1")
 					(unit 1)
 				)

Commit message: Added files for production & fixed some minor errors on the silkscreen
Parts:
- added SW1: SW_SPST, Button_Switch_THT:SW_TH_Tactile_Omron_B3F-102x, symbol Switch:SW_SPST
- U1: now left out of the parts list
- renumbered H2 to H1, H6 to H2, H5 to H3, H3 to H4, H4 to H5, H1 to H6
Connections:
- net GND: now also SW1.2 (B)
- net at U1.12 (D3): now also SW1.1 (A)
- no-connect marks 7 -> 6
Other:
- moved on the sheet: U1
